Commit message: Able to move and drive

File: description/robot.urdf.xacro (robot description, xacro)
@@ -2,3 +2,4 @@
 <robot xmlns:xacro="http://www.ros.org/wiki/xacro"  name="robot">
 <xacro:include filename="robot_core.xacro"/>
+<xacro:include filename="gazebo_control.xacro"/>
 </robot>

File: description/robot_core.xacro (robot description, xacro)
@@ -42,9 +42,14 @@
         </xacro:inertial_box>
     </link>
+    <gazebo reference = "chassis_link" >
+        <material>
+            Gazebo/White
+        </material>
+    </gazebo>
     <!--       LEFT WHEEL         -->
     <joint name="left_wheel_joint" type="continuous">
         <parent link="base_link"/>
         <child link="left_wheel_link"/>
-        <origin xyz="0.0 0.175 0.0" rpy="${pi/2} 0 0"/>
+        <origin xyz="0.0 -0.175 0.0" rpy="-${pi/2} 0 0"/>
         <axis xyz="0.0 0.0 1"/>
     </joint>
@@ -65,9 +70,14 @@
         </xacro:inertial_cylinder>
     </link>
+    <gazebo reference = "left_wheel_link" >
+        <material>
+            Gazebo/Blue
+        </material>
+    </gazebo>
     <!--        RIGHT WHEEL       -->
     <joint name="right_wheel_joint" type="continuous">
         <parent link="base_link"/>
         <child link="right_wheel_link"/>
-        <origin xyz="0.0 -0.175 0.0" rpy="-${pi/2} 0 0"/>
+        <origin xyz="0.0 0.175 0.0" rpy="${pi/2} 0 0"/>
         <axis xyz="0.0 0.0 -1"/>
     </joint>
@@ -88,4 +98,9 @@
         </xacro:inertial_cylinder>
     </link>
+    <gazebo reference = "right_wheel_link" >
+        <material>
+            Gazebo/Blue
+        </material>
+    </gazebo>
     <!--    CASTER WHEEL    -->
     <joint name="caster_wheel_joint" type="fixed">
@@ -110,3 +125,10 @@
         </xacro:inertial_sphere>
     </link>
+    <gazebo reference = "caster_wheel_link" >
+        <material>
+            Gazebo/Black
+        </material>
+        <mu1 value="0.001"/>
+        <mu2 value="0.001"/>
+    </gazebo>
 </robot>

Commit message: Camera and sensor added

File: description/robot.urdf.xacro (robot description, xacro)
@@ -3,3 +3,5 @@
 <xacro:include filename="robot_core.xacro"/>
 <xacro:include filename="gazebo_control.xacro"/>
+<xacro:include filename="lidar.xacro"/>
+<xacro:include filename="camera.xacro"/>
 </robot>

File: description/robot_core.xacro (robot description, xacro)
@@ -13,4 +13,7 @@
     <material name="black">
         <color rgba="0.0 0.0 0.0 1"/>
+    </material>
+    <material name="red">
+        <color rgba="1 0.0 0.0 1"/>
     </material>
     <!--         BASE LINK           -->
